Commit message: Update turtlebot3_flushbot.urdf.xacro

File: turtlebot3_description/urdf/turtlebot3_flushbot.urdf.xacro (robot description, xacro)
@@ -156,5 +156,5 @@
     <parent link="base_link"/>
     <child link="imu_link"/>
-    <origin xyz="0 0 0.0845" rpy="0 0 0"/>
+    <origin xyz="0.08 0.08 0.0845" rpy="0 0 0"/>
   </joint>
   <link name="imu_link"/>
@@ -162,10 +162,10 @@
     <parent link="base_link"/>
     <child link="base_scan"/>
-    <origin xyz="0.175 0 0.70" rpy="0 0 0"/>
+    <origin xyz="0.115 0.145 0.58" rpy="0 0 0"/>
   </joint>
 <!-- sensor place -->
   <link name="base_scan">
     <visual>
-      <origin xyz="0 0 0.0" rpy="0 0 0"/>
+      <origin xyz="0 0 0.0" rpy="0 0 3.141"/>
       <geometry>
         <mesh filename="package://turtlebot3_description/meshes/sensors/lds.stl" scale="0.001 0.001 0.001"/>
